File: sequencer.kicad_pcb (KiCad board)
At the start: 4 copper layers, 120 x 60 mm, 90 parts, among them J1 AudioJack2_SwitchT, J2 AudioJack2_SwitchT, J3 AudioJack2_SwitchT, J4 Conn_ARM_JTAG_SWD_10, J5 Conn_01x06_Male, J6 Conn_01x02_Male, SW1 OS102011MS2QN1, SW10 EG1206A, SW2 OS102011MS2QN1, SW3 OS102011MS2QN1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

Commit message: r0 fab
Parts:
- added LOGO1: CC-BY-SA_0.33in, Symbol_CreativeCommons:CC-BY-SA_SilkScreenTop_Small, B.Cu at (183.8, 78.8)
- added LOGO2: Logo_MadeWithKiCad, Symbol:KiCad-Logo2_5mm_SilkScreen, B.Cu at (170.0, 77.8)
- added LOGO3: Logo_Open_Hardware_Small, Symbol:OSHW-Logo2_7.3x6mm_SilkScreen, B.Cu at (170.2, 70.0)
- U2: value 74HC4051 -> 74HCT4051
Other:
- board text added: "JLCJLCJLCJLC"
